Commit message: updated youbot.urdf and srdf

File: urdf/youbot.urdf (robot description, URDF)
Before this commit: robot youbot, 21 links, 20 joints
Links:
- removed link caster_link_bl
- removed link caster_link_br
- removed link caster_link_fl
- removed link caster_link_fr
- removed link wheel_link_bl
- removed link wheel_link_br
- removed link wheel_link_fl
- removed link wheel_link_fr
- added link base_laser_rear_link, mass 0.16; collision mesh filename=package://youbot_description/meshes/sensors/hokuyo_convex.d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; visual mesh filename=package://youbot_description/meshes/sensors/hokuyo.dae
- added link tower_cam3d_camera, mass 0.01; collision mesh filename=package://youbot_robot_description/meshes/sensors/kinect.dae; visual mesh filename=package://youbot_robot_description/meshes/sensors/kinect.dae
- added link tower_cam3d_depth_frame, mass 0.01
- added link tower_cam3d_depth_optical_frame, mass 0.001
- added link tower_cam3d_rgb_frame, mass 0.001
- added link tower_cam3d_rgb_optical_frame, mass 0.001
- added link tower_link, mass 0.01; collision box size=0.03 0.03 0.49; visual box size=0.03 0.03 0.49
- link arm_link_0: geometry collision mesh filename=package://youbot_description/meshes/youbot_arm/arm0_convex.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; visual mesh filename=package://youbot_description/meshes/youbot_arm/arm0.dae
- link arm_link_1: geometry collision mesh filename=package://youbot_description/meshes/youbot_arm/arm1_convex.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; visual mesh filename=package://youbot_description/meshes/youbot_arm/arm1.dae
- link arm_link_2: geometry collision mesh filename=package://youbot_description/meshes/youbot_arm/arm2_convex.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; visual mesh filename=package://youbot_description/meshes/youbot_arm/arm2.dae
- link arm_link_3: geometry collision mesh filename=package://youbot_description/meshes/youbot_arm/arm3_convex.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; visual mesh filename=package://youbot_description/meshes/youbot_arm/arm3.dae
- link arm_link_4: geometry collision mesh filename=package://youbot_description/meshes/youbot_arm/arm4_convex.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; visual mesh filename=package://youbot_description/meshes/youbot_arm/arm4.dae
- link arm_link_5: geometry collision mesh filename=package://youbot_description/meshes/youbot_arm/arm5_convex.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; visual mesh filename=package://youbot_description/meshes/youbot_arm/arm5.dae
- link base_laser_front_link: geometry collision mesh filename=package://youbot_description/meshes/sensors/hokuyo_convex.d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; visual mesh filename=package://youbot_description/meshes/sensors/hokuyo.dae
- link base_link: geometry collision mesh filename=package://youbot_description/meshes/youbot_base/base_convex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; visual mesh filename=package://youbot_description/meshes/youbot_base/base.dae
- link gripper_finger_link_l: geometry collision mesh filename=package://youbot_description/meshes/youbot_gripper/finger_c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; visual mesh filename=package://youbot_description/meshes/youbot_gripper/finger.d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
- link gripper_finger_link_r: geometry collision mesh filename=package://youbot_description/meshes/youbot_gripper/finger_c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; visual mesh filename=package://youbot_description/meshes/youbot_gripper/finger.d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
- link gripper_palm_link: mass 0.75 -> 0.1; geometry collision mesh filename=package://youbot_description/meshes/youbot_gripper/palm_con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; visual mesh filename=package://youbot_description/meshes/youbot_gripper/palm.dae
- link plate_link: geometry collision mesh filename=package://youbot_description/meshes/youbot_plate/plate_conv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; visual mesh filename=package://youbot_description/meshes/youbot_plate/plate.dae
Joints:
- removed joint caster_joint_bl
- removed joint caster_joint_br
- removed joint caster_joint_fl
- removed joint caster_joint_fr
- removed joint wheel_joint_bl
- removed joint wheel_joint_br
- removed joint wheel_joint_fl
- removed joint wheel_joint_fr
- added joint base_laser_rear_hokuyo_urg04_laser_joint: type fixed, parent base_link, child base_laser_rear_link, origin xyz=-0.3 0.0 -0.03 rpy=0 0 3.14159265359, axis 0 1 0
- added joint tower_cam3d_camera_depth_joint: type fixed, parent tower_cam3d_camera, child tower_cam3d_depth_frame, origin xyz=0 0.018 0 rpy=0 0 0
- added joint tower_cam3d_camera_depth_optical_joint: type fixed, parent tower_cam3d_depth_frame, child tower_cam3d_depth_optical_frame, origin xyz=0 0 0 rpy=-1.57079632679 0 -1.57079632679
- added joint tower_cam3d_camera_joint: type fixed, parent tower_link, child tower_cam3d_camera, origin xyz=0.0509 -0.03 0.49 rpy=0.0 0.545 0.0
- added joint tower_cam3d_camera_rgb_joint: type fixed, parent tower_cam3d_camera, child tower_cam3d_rgb_frame, origin xyz=0 -0.005 0 rpy=0 0 0
- added joint tower_cam3d_camera_rgb_optical_joint: type fixed, parent tower_cam3d_rgb_frame, child tower_cam3d_rgb_optical_frame, origin xyz=0 0 0 rpy=-1.57079632679 0 -1.57079632679
- added joint tower_joint: type fixed, parent plate_link, child tower_link, origin xyz=-0.0659 0.0 0.025 rpy=0 0 0
- joint arm_joint_1: axis 0 0 1 -> 0 0 -1; limit lower=0 upper=5.89921287174 effort=10 velocity=1.57079632679 -> lower=0 upper=5.89921287174 effort=9.5 velocity=1.57079632679; origin xyz=0.024 0 0.096 rpy=0 0 0 -> xyz=0.024 0 0.096 rpy=0 0 2.96705972839
- joint arm_joint_2: axis 0 -1 0 -> 0 1 0; limit lower=0 upper=2.70526034059 effort=10 velocity=1.57079632679 -> lower=0 upper=2.70526034059 effort=9.5 velocity=1.57079632679; origin xyz=0.033 0 0.019 rpy=0 0 0 -> xyz=0.033 0 0.019 rpy=0 -1.1344640138 0
- joint arm_joint_3: limit lower=-5.18362787842 upper=0 effort=10 velocity=1.57079632679 -> lower=-5.18362787842 upper=0 effort=6.0 velocity=1.57079632679; origin xyz=0.000 0.000 0.155 rpy=0 0 0 -> xyz=0.000 0.000 0.155 rpy=0 2.54818070791 0
- joint arm_joint_4: axis 0 -1 0 -> 0 1 0; limit lower=0 upper=3.57792496659 effort=10 velocity=1.57079632679 -> lower=0 upper=3.57792496659 effort=2.0 velocity=1.57079632679; origin xyz=0.000 0.000 0.135 rpy=0 0 0 -> xyz=0.000 0.000 0.135 rpy=0 -1.78896248329 0
- joint arm_joint_5: axis 0 0 1 -> 0 0 -1; limit lower=0 upper=5.84685299418 effort=10 velocity=1.57079632679 -> lower=0 upper=5.84685299418 effort=1 velocity=1.57079632679; origin xyz=-0.002 0 0.130 rpy=0 0 0 -> xyz=-0.002 0 0.130 rpy=0 0 2.92342649709
- joint gripper_finger_joint_l: type fixed -> prismatic
- joint gripper_finger_joint_r: type fixed -> prismatic
