Commit message: Working collision component in sim for ring 5 in ur5

File: urdf/skin_sim.urdf.xacro (robot description, xacro)
@@ -27,7 +27,7 @@
 	  <parent link="forearm_link"/>
 	  <child link="forerarm_skin_root_cell_link"/>
-	  <origin xyz="0.0 0.0 0.0" rpy="0.  0.  0."/>
-          <axis xyz="0 0 1" />
-          <limit lower="0" upper="0" effort="150.0" velocity="3.15"/>
+	  <origin xyz="-0.003 -0.05 0.32" rpy="1.57  1.57  0."/>
+          <axis xyz="0 0 1" />
+          <limit lower="${-pi}" upper="${pi}" effort="150.0" velocity="3.15"/>
 </joint>
 <link name="forerarm_skin_link_0">
@@ -48,7 +48,8 @@
 	  <parent link="forerarm_skin_root_cell_link"/>
 	  <child link="forerarm_skin_link_0"/>
-	  <origin xyz="-0.02313 0.03352 0.23674" rpy="2.83297311  -1.54208643 2.44288303"/>
-          <axis xyz="0 0 1" />
-          <limit lower="0" upper="0" effort="150.0" velocity="3.15"/>
+<!--  <origin xyz="0.122545 0.0452926 -0.0396807" rpy="1.46  0.01 -0."/> -->
+	  <origin xyz="0.122545 0.0452926 -0.0396807" rpy="4.79  0.07 -0."/>
+          <axis xyz="0 0 1" />
+          <limit lower="${-pi}" upper="${pi}" effort="150.0" velocity="3.15"/>
 </joint>
 <link name="forerarm_skin_link_1">
@@ -69,7 +70,8 @@
 	  <parent link="forerarm_skin_root_cell_link"/>
 	  <child link="forerarm_skin_link_1"/>
-	  <origin xyz="-0.04032 -0.015129 0.23696" rpy="1.06341521  -1.48901494 -0.78506072"/>
-          <axis xyz="0 0 1" />
-          <limit lower="0" upper="0" effort="150.0" velocity="3.15"/>
+<!-- <origin xyz="0.122971 0.0347329 -0.0140614" rpy="0.88  0.03 -0."/> -->
+	  <origin xyz="0.122971 0.0347329 -0.0140614" rpy="5.35  0.07 -0."/>
+          <axis xyz="0 0 1" />
+          <limit lower="${-pi}" upper="${pi}" effort="150.0" velocity="3.15"/>
 </joint>
 <link name="forerarm_skin_link_2">
@@ -90,7 +92,7 @@
 	  <parent link="forerarm_skin_root_cell_link"/>
 	  <child link="forerarm_skin_link_2"/>
-	  <origin xyz="-0.0254929 -0.0339481 0.2358651" rpy="2.262972 -1.487026 -1.356827"/>
-          <axis xyz="0 0 1" />
-          <limit lower="0" upper="0" effort="150.0" velocity="3.15"/>
+	  <origin xyz="0.121427 0.0122404 -0.00364349" rpy="0.25  0.05  0."/>
+          <axis xyz="0 0 1" />
+          <limit lower="${-pi}" upper="${pi}" effort="150.0" velocity="3.15"/>
 </joint>
 <link name="forerarm_skin_link_3">
@@ -111,7 +113,7 @@
 	  <parent link="forerarm_skin_root_cell_link"/>
 	  <child link="forerarm_skin_link_3"/>
-	  <origin xyz="0.0004 -0.0441 0.23518" rpy="0.2035706 -1.5367411 1.35411575"/>
-          <axis xyz="0 0 1" />
-          <limit lower="0" upper="0" effort="150.0" velocity="3.15"/>
+	  <origin xyz="0.120852 -0.0153018 -0.00418709" rpy="0.3   0.05  0."/>
+          <axis xyz="0 0 1" />
+          <limit lower="${-pi}" upper="${pi}" effort="150.0" velocity="3.15"/>
 </joint>
 <link name="forerarm_skin_link_4">
@@ -132,7 +134,7 @@
 	  <parent link="forerarm_skin_root_cell_link"/>
 	  <child link="forerarm_skin_link_4"/>
-	  <origin xyz="0.026086 0.03677 0.23527" rpy="-2.34960077 -1.49847097 -1.75719079"/>
-          <axis xyz="0 0 1" />
-          <limit lower="0" upper="0" effort="150.0" velocity="3.15"/>
+	  <origin xyz="0.119741 -0.0385305 -0.0190389" rpy="0.83 -0.04 -0."/>
+          <axis xyz="0 0 1" />
+          <limit lower="${-pi}" upper="${pi}" effort="150.0" velocity="3.15"/>
 </joint>
 <link name="forerarm_skin_link_5">
@@ -153,7 +155,7 @@
 	  <parent link="forerarm_skin_root_cell_link"/>
 	  <child link="forerarm_skin_link_5"/>
-	  <origin xyz="0.04277 -0.01486 0.23704" rpy="-2.16054646 -1.50515821 -1.31557256"/>
-          <axis xyz="0 0 1" />
-          <limit lower="0" upper="0" effort="150.0" velocity="3.15"/>
+	  <origin xyz="0.119756 -0.0512256 -0.0430332" rpy="1.52  0.   -0."/>
+          <axis xyz="0 0 1" />
+          <limit lower="${-pi}" upper="${pi}" effort="150.0" velocity="3.15"/>
 </joint>
 <link name="forerarm_skin_link_6">
@@ -174,7 +176,7 @@
 	  <parent link="forerarm_skin_root_cell_link"/>
 	  <child link="forerarm_skin_link_6"/>
-	  <origin xyz="0.04285 0.01209 0.2382" rpy="-2.17682483 -1.51293455 -0.67460558"/>
-          <axis xyz="0 0 1" />
-          <limit lower="0" upper="0" effort="150.0" velocity="3.15"/>
+	  <origin xyz="0.118712 -0.0446355 -0.0687232" rpy="2.02  0.    0."/>
+          <axis xyz="0 0 1" />
+          <limit lower="${-pi}" upper="${pi}" effort="150.0" velocity="3.15"/>
 </joint>
 <link name="forerarm_skin_link_7">
@@ -195,7 +197,72 @@
 	  <parent link="forerarm_skin_root_cell_link"/>
 	  <child link="forerarm_skin_link_7"/>
-	  <origin xyz="0.02665 0.03505 0.23515" rpy="0.99763746 -1.51906704 3.11362853"/>
-          <axis xyz="0 0 1" />
-          <limit lower="0" upper="0" effort="150.0" velocity="3.15"/>
+	  <origin xyz="0.119505 -0.0267679 -0.0889594" rpy="2.55 -0.02 -0."/>
+          <axis xyz="0 0 1" />
+          <limit lower="${-pi}" upper="${pi}" effort="150.0" velocity="3.15"/>
+</joint>
+<link name="forerarm_skin_link_8">
+ 	<visual>
+	      <geometry>
+		<sphere radius="0.005"/>
+	      </geometry>
+	      <material name="white"/>
+	</visual>
+	<collision>
+  	<origin xyz="0 0 0" rpy="0 0 0" />
+    	<geometry>
+    	    <sphere radius="0.005"/>
+        </geometry>
+  </collision>
+</link>
+<joint name="forerarm_skin_cell_joint_8" type="revolute">
+	  <parent link="forerarm_skin_root_cell_link"/>
+	  <child link="forerarm_skin_link_8"/>
+	  <origin xyz="0.119639 -0.00112243 -0.0964335" rpy="3.11  0.07 -0."/>
+          <axis xyz="0 0 1" />
+          <limit lower="${-pi}" upper="${pi}" effort="150.0" velocity="3.15"/>
+</joint>
+<link name="forerarm_skin_link_9">
+ 	<visual>
+	      <geometry>
+		<sphere radius="0.005"/>
+	      </geometry>
+	      <material name="white"/>
+	</visual>
+	<collision>
+  	<origin xyz="0 0 0" rpy="0 0 0" />
+    	<geometry>
+    	    <sphere radius="0.005"/>
+        </geometry>
+  </collision>
+</link>
+<joint name="forerarm_skin_cell_joint_9" type="revolute">
+	  <parent link="forerarm_skin_root_cell_link"/>
+	  <child link="forerarm_skin_link_9"/>
+<!--  <origin xyz="0.120033 0.0253832 -0.088699" rpy="2.48  0.02 -0."/>-->
+	  <origin xyz="0.120033 0.0253832 -0.088699" rpy="3.67  0.07 -0."/>
+          <axis xyz="0 0 1" />
+          <limit lower="${-pi}" upper="${pi}" effort="150.0" velocity="3.15"/>
+</joint>
+<link name="forerarm_skin_link_10">
+ 	<visual>
+	      <geometry>
+		<sphere radius="0.005"/>
+	      </geometry>
+	      <material name="white"/>
+	</visual>
+	<collision>
+  	<origin xyz="0 0 0" rpy="0 0 0" />
+    	<geometry>
+    	    <sphere radius="0.005"/>
+        </geometry>
+  </collision>
+</link>
+<joint name="forerarm_skin_cell_joint_10" type="revolute">
+	  <parent link="forerarm_skin_root_cell_link"/>
+	  <child link="forerarm_skin_link_10"/>
+<!--  <o<origin xyz="0.122276 0.0426263 -0.0664088" rpy="1.97  0.   -0."/> -->
+	  <origin xyz="0.122276 0.0426263 -0.0664088" rpy="4.23  0.07 -0."/>
+          <axis xyz="0 0 1" />
+          <limit lower="${-pi}" upper="${pi}" effort="150.0" velocity="3.15"/>
 </joint>
 <!--Finishers-->

File: urdf/ur5_robot_with_ring_forearm_sim.urdf (robot description, URDF)
Before this commit: robot ur5, 20 links, 19 joints
Links:
- added link forerarm_skin_link_10; collision sphere radius=0.005; visual sphere radius=0.005
- added link forerarm_skin_link_8; collision sphere radius=0.005; visual sphere radius=0.005
- added link forerarm_skin_link_9; collision sphere radius=0.005; visual sphere radius=0.005
Joints:
- added joint forerarm_skin_cell_joint_10: type revolute, parent forerarm_skin_root_cell_link, child forerarm_skin_link_10, origin xyz=0.122276 0.0426263 -0.0664088 rpy=4.23  0.07 -0., axis 0 0 1, limit lower=-3.14159265 upper=3.14159265 effort=150.0 velocity=3.15
- added joint forerarm_skin_cell_joint_8: type revolute, parent forerarm_skin_root_cell_link, child forerarm_skin_link_8, origin xyz=0.119639 -0.00112243 -0.0964335 rpy=3.11  0.07 -0., axis 0 0 1, limit lower=-3.14159265 upper=3.14159265 effort=150.0 velocity=3.15
- added joint forerarm_skin_cell_joint_9: type revolute, parent forerarm_skin_root_cell_link, child forerarm_skin_link_9, origin xyz=0.120033 0.0253832 -0.088699 rpy=3.67  0.07 -0., axis 0 0 1, limit lower=-3.14159265 upper=3.14159265 effort=150.0 velocity=3.15
- joint forerarm_skin_cell_joint_0: origin xyz=-0.02313 0.03352 0.23674 rpy=2.83297311  -1.54208643 2.44288303 -> xyz=0.122545 0.0452926 -0.0396807 rpy=4.79  0.07 -0.
- joint forerarm_skin_cell_joint_1: origin xyz=-0.04032 -0.015129 0.23696 rpy=1.06341521  -1.48901494 -0.78506072 -> xyz=0.122971 0.0347329 -0.0140614 rpy=5.35  0.07 -0.
- joint forerarm_skin_cell_joint_2: origin xyz=-0.0254929 -0.0339481 0.2358651 rpy=2.262972 -1.487026 -1.356827 -> xyz=0.121427 0.0122404 -0.00364349 rpy=0.25  0.05  0.
- joint forerarm_skin_cell_joint_3: origin xyz=0.0004 -0.0441 0.23518 rpy=0.2035706 -1.5367411 1.35411575 -> xyz=0.120852 -0.0153018 -0.00418709 rpy=0.3   0.05  0.
- joint forerarm_skin_cell_joint_4: origin xyz=0.026086 0.03677 0.23527 rpy=-2.34960077 -1.49847097 -1.75719079 -> xyz=0.119741 -0.0385305 -0.0190389 rpy=0.83 -0.04 -0.
- joint forerarm_skin_cell_joint_5: origin xyz=0.04277 -0.01486 0.23704 rpy=-2.16054646 -1.50515821 -1.31557256 -> xyz=0.119756 -0.0512256 -0.0430332 rpy=1.52  0.   -0.
- joint forerarm_skin_cell_joint_6: origin xyz=0.04285 0.01209 0.2382 rpy=-2.17682483 -1.51293455 -0.67460558 -> xyz=0.118712 -0.0446355 -0.0687232 rpy=2.02  0.    0.
- joint forerarm_skin_cell_joint_7: origin xyz=0.02665 0.03505 0.23515 rpy=0.99763746 -1.51906704 3.11362853 -> xyz=0.119505 -0.0267679 -0.0889594 rpy=2.55 -0.02 -0.
- joint forerarm_skin_root_cell_joint: limit lower=0 upper=0 effort=150.0 velocity=3.15 -> lower=-3.14159265 upper=3.14159265 effort=150.0 velocity=3.15; origin xyz=0.0 0.0 0.0 rpy=0.  0.  0. -> xyz=-0.003 -0.05 0.32 rpy=1.57  1.57  0.
