Commit message: Added 4th ring to urdf.

File: urdf/skin.urdf.xacro (robot description, xacro)
@@ -4,9 +4,10 @@
        xmlns:interface="http://playerstage.sourceforge.net/gazebo/xmlschema/#interface"
        xmlns:xacro="http://ros.org/wiki/xacro">
-	<!--Common definitions
-	<xacro:include filename="$(find tom_description)/urdf/common.xacro"/>-->
+	<!--Common definitions -->
+	<xacro:include filename="$(find tom_description)/urdf/common.xacro"/>
 	<!-- xacro sensors  -->
 	<xacro:macro name="skin" params="name">
-<link name="forerarm_skin_root_cell_link">
+<!-- FOREARM -->
+<link name="forearm_skin_root_cell_link">
  	<visual>
 	      <geometry>
@@ -24,180 +25,343 @@
   </collision>
 </link>
-<joint name="forerarm_skin_root_cell_joint" type="fixed">
+<joint name="forearm_skin_root_cell_joint" type="fixed">
 	  <parent link="forearm_link"/>
-	  <child link="forerarm_skin_root_cell_link"/>
+	  <child link="forearm_skin_root_cell_link"/>
 	  <origin xyz="0.0 0.0 0.0" rpy="0.  0.  0."/>
           <axis xyz="0 0 1" />
           <limit lower="0" upper="0" effort="150.0" velocity="3.15"/>
 </joint>
-<link name="forerarm_skin_link_0">
- 	<visual>
-	      <geometry>
-		<sphere radius="0.005"/>
-	      </geometry>
-	      <material name="white"/>
-	</visual>
-	<collision>
-  	<origin xyz="0 0 0" rpy="0 0 0" />
-    	<geometry>
-    	    <sphere radius="0.005"/>
-        </geometry>
-  </collision>
-</link>
-<joint name="forerarm_skin_cell_joint_0" type="revolute">
-	  <parent link="forerarm_skin_root_cell_link"/>
-	  <child link="forerarm_skin_link_0"/>
+<link name="forearm_ring_5_link_0">
+ 	<visual>
+	      <geometry>
+		<sphere radius="0.005"/>
+	      </geometry>
+	      <material name="white"/>
+	</visual>
+	<collision>
+  	<origin xyz="0 0 0" rpy="0 0 0" />
+    	<geometry>
+    	    <sphere radius="0.005"/>
+        </geometry>
+  </collision>
+</link>
+<joint name="forearm_ring_5_joint_0" type="fixed">
+	  <parent link="forearm_skin_root_cell_link"/>
+	  <child link="forearm_ring_5_link_0"/>
 	  <origin xyz="-0.02313 0.03352 0.23674" rpy="2.83297311  -1.54208643 2.44288303"/>
           <axis xyz="0 0 1" />
           <limit lower="0" upper="0" effort="150.0" velocity="3.15"/>
 </joint>
-<link name="forerarm_skin_link_1">
- 	<visual>
-	      <geometry>
-		<sphere radius="0.005"/>
-	      </geometry>
-	      <material name="white"/>
-	</visual>
-	<collision>
-  	<origin xyz="0 0 0" rpy="0 0 0" />
-    	<geometry>
-    	    <sphere radius="0.005"/>
-        </geometry>
-  </collision>
-</link>
-<joint name="forerarm_skin_cell_joint_1" type="revolute">
-	  <parent link="forerarm_skin_root_cell_link"/>
-	  <child link="forerarm_skin_link_1"/>
+<link name="forearm_ring_5_link_1">
+ 	<visual>
+	      <geometry>
+		<sphere radius="0.005"/>
+	      </geometry>
+	      <material name="white"/>
+	</visual>
+	<collision>
+  	<origin xyz="0 0 0" rpy="0 0 0" />
+    	<geometry>
+    	    <sphere radius="0.005"/>
+        </geometry>
+  </collision>
+</link>
+<joint name="forearm_ring_5_joint_1" type="fixed">
+	  <parent link="forearm_skin_root_cell_link"/>
+	  <child link="forearm_ring_5_link_1"/>
 	  <origin xyz="-0.04032 -0.015129 0.23696" rpy="1.06341521  -1.48901494 -0.78506072"/>
           <axis xyz="0 0 1" />
           <limit lower="0" upper="0" effort="150.0" velocity="3.15"/>
 </joint>
-<link name="forerarm_skin_link_2">
- 	<visual>
-	      <geometry>
-		<sphere radius="0.005"/>
-	      </geometry>
-	      <material name="white"/>
-	</visual>
-	<collision>
-  	<origin xyz="0 0 0" rpy="0 0 0" />
-    	<geometry>
-    	    <sphere radius="0.005"/>
-        </geometry>
-  </collision>
-</link>
-<joint name="forerarm_skin_cell_joint_2" type="revolute">
-	  <parent link="forerarm_skin_root_cell_link"/>
-	  <child link="forerarm_skin_link_2"/>
+<link name="forearm_ring_5_link_2">
+ 	<visual>
+	      <geometry>
+		<sphere radius="0.005"/>
+	      </geometry>
+	      <material name="white"/>
+	</visual>
+	<collision>
+  	<origin xyz="0 0 0" rpy="0 0 0" />
+    	<geometry>
+    	    <sphere radius="0.005"/>
+        </geometry>
+  </collision>
+</link>
+<joint name="forearm_ring_5_joint_2" type="fixed">
+	  <parent link="forearm_skin_root_cell_link"/>
+	  <child link="forearm_ring_5_link_2"/>
 	  <origin xyz="-0.0254929 -0.0339481 0.2358651" rpy="2.262972 -1.487026 -1.356827"/>
           <axis xyz="0 0 1" />
           <limit lower="0" upper="0" effort="150.0" velocity="3.15"/>
 </joint>
-<link name="forerarm_skin_link_3">
- 	<visual>
-	      <geometry>
-		<sphere radius="0.005"/>
-	      </geometry>
-	      <material name="white"/>
-	</visual>
-	<collision>
-  	<origin xyz="0 0 0" rpy="0 0 0" />
-    	<geometry>
-    	    <sphere radius="0.005"/>
-        </geometry>
-  </collision>
-</link>
-<joint name="forerarm_skin_cell_joint_3" type="revolute">
-	  <parent link="forerarm_skin_root_cell_link"/>
-	  <child link="forerarm_skin_link_3"/>
+<link name="forearm_ring_5_link_3">
+ 	<visual>
+	      <geometry>
+		<sphere radius="0.005"/>
+	      </geometry>
+	      <material name="white"/>
+	</visual>
+	<collision>
+  	<origin xyz="0 0 0" rpy="0 0 0" />
+    	<geometry>
+    	    <sphere radius="0.005"/>
+        </geometry>
+  </collision>
+</link>
+<joint name="forearm_ring_5_joint_3" type="fixed">
+	  <parent link="forearm_skin_root_cell_link"/>
+	  <child link="forearm_ring_5_link_3"/>
 	  <origin xyz="0.0004 -0.0441 0.23518" rpy="0.2035706 -1.5367411 1.35411575"/>
           <axis xyz="0 0 1" />
           <limit lower="0" upper="0" effort="150.0" velocity="3.15"/>
 </joint>
-<link name="forerarm_skin_link_4">
- 	<visual>
-	      <geometry>
-		<sphere radius="0.005"/>
-	      </geometry>
-	      <material name="white"/>
-	</visual>
-	<collision>
-  	<origin xyz="0 0 0" rpy="0 0 0" />
-    	<geometry>
-    	    <sphere radius="0.005"/>
-        </geometry>
-  </collision>
-</link>
-<joint name="forerarm_skin_cell_joint_4" type="revolute">
-	  <parent link="forerarm_skin_root_cell_link"/>
-	  <child link="forerarm_skin_link_4"/>
-	  <origin xyz="0.026086 0.03677 0.23527" rpy="-2.34960077 -1.49847097 -1.75719079"/>
-          <axis xyz="0 0 1" />
-          <limit lower="0" upper="0" effort="150.0" velocity="3.15"/>
-</joint>
-<link name="forerarm_skin_link_5">
- 	<visual>
-	      <geometry>
-		<sphere radius="0.005"/>
-	      </geometry>
-	      <material name="white"/>
-	</visual>
-	<collision>
-  	<origin xyz="0 0 0" rpy="0 0 0" />
-    	<geometry>
-    	    <sphere radius="0.005"/>
-        </geometry>
-  </collision>
-</link>
-<joint name="forerarm_skin_cell_joint_5" type="revolute">
-	  <parent link="forerarm_skin_root_cell_link"/>
-	  <child link="forerarm_skin_link_5"/>
+<link name="forearm_ring_5_link_4">
+ 	<visual>
+	      <geometry>
+		<sphere radius="0.005"/>
+	      </geometry>
+	      <material name="white"/>
+	</visual>
+	<collision>
+  	<origin xyz="0 0 0" rpy="0 0 0" />
+    	<geometry>
+    	    <sphere radius="0.005"/>
+        </geometry>
+  </collision>
+</link>
+<joint name="forearm_ring_5_joint_4" type="fixed">
+	  <parent link="forearm_skin_root_cell_link"/>
+	  <child link="forearm_ring_5_link_4"/>
+	  <origin xyz="0.026086 -0.03677 0.23527" rpy="-2.34960077 -1.49847097 -1.75719079"/>
+          <axis xyz="0 0 1" />
+          <limit lower="0" upper="0" effort="150.0" velocity="3.15"/>
+</joint>
+<link name="forearm_ring_5_link_5">
+ 	<visual>
+	      <geometry>
+		<sphere radius="0.005"/>
+	      </geometry>
+	      <material name="white"/>
+	</visual>
+	<collision>
+  	<origin xyz="0 0 0" rpy="0 0 0" />
+    	<geometry>
+    	    <sphere radius="0.005"/>
+        </geometry>
+  </collision>
+</link>
+<joint name="forearm_ring_5_joint_5" type="fixed">
+	  <parent link="forearm_skin_root_cell_link"/>
+	  <child link="forearm_ring_5_link_5"/>
 	  <origin xyz="0.04277 -0.01486 0.23704" rpy="-2.16054646 -1.50515821 -1.31557256"/>
           <axis xyz="0 0 1" />
           <limit lower="0" upper="0" effort="150.0" velocity="3.15"/>
 </joint>
-<link name="forerarm_skin_link_6">
- 	<visual>
-	      <geometry>
-		<sphere radius="0.005"/>
-	      </geometry>
-	      <material name="white"/>
-	</visual>
-	<collision>
-  	<origin xyz="0 0 0" rpy="0 0 0" />
-    	<geometry>
-    	    <sphere radius="0.005"/>
-        </geometry>
-  </collision>
-</link>
-<joint name="forerarm_skin_cell_joint_6" type="revolute">
-	  <parent link="forerarm_skin_root_cell_link"/>
-	  <child link="forerarm_skin_link_6"/>
+<link name="forearm_ring_5_link_6">
+ 	<visual>
+	      <geometry>
+		<sphere radius="0.005"/>
+	      </geometry>
+	      <material name="white"/>
+	</visual>
+	<collision>
+  	<origin xyz="0 0 0" rpy="0 0 0" />
+    	<geometry>
+    	    <sphere radius="0.005"/>
+        </geometry>
+  </collision>
+</link>
+<joint name="forearm_ring_5_joint_6" type="fixed">
+	  <parent link="forearm_skin_root_cell_link"/>
+	  <child link="forearm_ring_5_link_6"/>
 	  <origin xyz="0.04285 0.01209 0.2382" rpy="-2.17682483 -1.51293455 -0.67460558"/>
           <axis xyz="0 0 1" />
           <limit lower="0" upper="0" effort="150.0" velocity="3.15"/>
 </joint>
-<link name="forerarm_skin_link_7">
- 	<visual>
-	      <geometry>
-		<sphere radius="0.005"/>
-	      </geometry>
-	      <material name="white"/>
-	</visual>
-	<collision>
-  	<origin xyz="0 0 0" rpy="0 0 0" />
-    	<geometry>
-    	    <sphere radius="0.005"/>
-        </geometry>
-  </collision>
-</link>
-<joint name="forerarm_skin_cell_joint_7" type="revolute">
-	  <parent link="forerarm_skin_root_cell_link"/>
-	  <child link="forerarm_skin_link_7"/>
+<link name="forearm_ring_5_link_7">
+ 	<visual>
+	      <geometry>
+		<sphere radius="0.005"/>
+	      </geometry>
+	      <material name="white"/>
+	</visual>
+	<collision>
+  	<origin xyz="0 0 0" rpy="0 0 0" />
+    	<geometry>
+    	    <sphere radius="0.005"/>
+        </geometry>
+  </collision>
+</link>
+<joint name="forearm_ring_5_joint_7" type="fixed">
+	  <parent link="forearm_skin_root_cell_link"/>
+	  <child link="forearm_ring_5_link_7"/>
 	  <origin xyz="0.02665 0.03505 0.23515" rpy="0.99763746 -1.51906704 3.11362853"/>
           <axis xyz="0 0 1" />
           <limit lower="0" upper="0" effort="150.0" velocity="3.15"/>
 </joint>
+<!-- NEW INFO-->
+<link name="forearm_ring_4_link_0">
+ 	<visual>
+	      <geometry>
+		<sphere radius="0.005"/>
+	      </geometry>
+	      <material name="white"/>
+	</visual>
+	<collision>
+  	<origin xyz="0 0 0" rpy="0 0 0" />
+    	<geometry>
+    	    <sphere radius="0.005"/>
+        </geometry>
+  </collision>
+</link>
+<joint name="forearm_ring_4_joint_0" type="fixed">
+	  <parent link="forearm_skin_root_cell_link"/>
+	  <child link="forearm_ring_4_link_0"/>
+	  <origin xyz="0.0147 0.0418 0.211" rpy="-0.2630 -1.4924 -1.5854"/>
+          <axis xyz="0 0 1" />
+          <limit lower="0" upper="0" effort="150.0" velocity="3.15"/>
+</joint>
+<link name="forearm_ring_4_link_1">
+ 	<visual>
+	      <geometry>
+		<sphere radius="0.005"/>
+	      </geometry>
+	      <material name="white"/>
+	</visual>
+	<collision>
+  	<origin xyz="0 0 0" rpy="0 0 0" />
+    	<geometry>
+    	    <sphere radius="0.005"/>
+        </geometry>
+  </collision>
+</link>
+<joint name="forearm_ring_4_joint_1" type="fixed">
+	  <parent link="forearm_skin_root_cell_link"/>
+	  <child link="forearm_ring_4_link_1"/>
+	  <origin xyz="0.0349 0.0252 0.2104" rpy="0.8048 -1.5595 2.9517"/>
+          <axis xyz="0 0 1" />
+          <limit lower="0" upper="0" effort="150.0" velocity="3.15"/>
+</joint>
+<link name="forearm_ring_4_link_2">
+ 	<visual>
+	      <geometry>
+		<sphere radius="0.005"/>
+	      </geometry>
+	      <material name="white"/>
+	</visual>
+	<collision>
+  	<origin xyz="0 0 0" rpy="0 0 0" />
+    	<geometry>
+    	    <sphere radius="0.005"/>
+        </geometry>
+  </collision>
+</link>
+<joint name="forearm_ring_4_joint_2" type="fixed">
+	  <parent link="forearm_skin_root_cell_link"/>
+	  <child link="forearm_ring_4_link_2"/>
+	  <origin xyz=" 0.0439 -0.0003 0.2101" rpy="0.9567 -1.542 2.211"/>
+          <axis xyz="0 0 1" />
+          <limit lower="0" upper="0" effort="150.0" velocity="3.15"/>
+</joint>
+<link name="forearm_ring_4_link_3">
+ 	<visual>
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
File: urdf/ur5_robot_with_ring_forearm.urdf (robot description, URDF)
Before this commit: robot ur5, 20 links, 19 joints
Links:
- removed link forerarm_skin_link_0
- removed link forerarm_skin_link_1
- removed link forerarm_skin_link_2
- removed link forerarm_skin_link_3
- removed link forerarm_skin_link_4
- removed link forerarm_skin_link_5
- removed link forerarm_skin_link_6
- removed link forerarm_skin_link_7
- removed link forerarm_skin_root_cell_link
- added link forearm_ring_4_link_0; collision sphere radius=0.005; visual sphere radius=0.005
- added link forearm_ring_4_link_1; collision sphere radius=0.005; visual sphere radius=0.005
- added link forearm_ring_4_link_2; collision sphere radius=0.005; visual sphere radius=0.005
- added link forearm_ring_4_link_3; collision sphere radius=0.005; visual sphere radius=0.005
- added link forearm_ring_4_link_4; collision sphere radius=0.005; visual sphere radius=0.005
- added link forearm_ring_4_link_5; collision sphere radius=0.005; visual sphere radius=0.005
- added link forearm_ring_4_link_6; collision sphere radius=0.005; visual sphere radius=0.005
- added link forearm_ring_4_link_7; collision sphere radius=0.005; visual sphere radius=0.005
- added link forearm_ring_5_link_0; collision sphere radius=0.005; visual sphere radius=0.005
- added link forearm_ring_5_link_1; collision sphere radius=0.005; visual sphere radius=0.005
- added link forearm_ring_5_link_2; collision sphere radius=0.005; visual sphere radius=0.005
- added link forearm_ring_5_link_3; collision sphere radius=0.005; visual sphere radius=0.005
- added link forearm_ring_5_link_4; collision sphere radius=0.005; visual sphere radius=0.005
- added link forearm_ring_5_link_5; collision sphere radius=0.005; visual sphere radius=0.005
- added link forearm_ring_5_link_6; collision sphere radius=0.005; visual sphere radius=0.005
- added link forearm_ring_5_link_7; collision sphere radius=0.005; visual sphere radius=0.005
- added link forearm_skin_root_cell_link; collision sphere radius=0.00000001; visual sphere radius=0.000001
Joints:
- removed joint forerarm_skin_cell_joint_0
- removed joint forerarm_skin_cell_joint_1
- removed joint forerarm_skin_cell_joint_2
- removed joint forerarm_skin_cell_joint_3
- removed joint forerarm_skin_cell_joint_4
- removed joint forerarm_skin_cell_joint_5
- removed joint forerarm_skin_cell_joint_6
- removed joint forerarm_skin_cell_joint_7
- removed joint forerarm_skin_root_cell_joint
- added joint forearm_ring_4_joint_0: type fixed, parent forearm_skin_root_cell_link, child forearm_ring_4_link_0, origin xyz=0.0147 0.0418 0.211 rpy=-0.2630 -1.4924 -1.5854, axis 0 0 1, limit lower=0 upper=0 effort=150.0 velocity=3.15
- added joint forearm_ring_4_joint_1: type fixed, parent forearm_skin_root_cell_link, child forearm_ring_4_link_1, origin xyz=0.0349 0.0252 0.2104 rpy=0.8048 -1.5595 2.9517, axis 0 0 1, limit lower=0 upper=0 effort=150.0 velocity=3.15
- added joint forearm_ring_4_joint_2: type fixed, parent forearm_skin_root_cell_link, child forearm_ring_4_link_2, origin xyz= 0.0439 -0.0003 0.2101 rpy=0.9567 -1.542 2.211, axis 0 0 1, limit lower=0 upper=0 effort=150.0 velocity=3.15
- added joint forearm_ring_4_joint_3: type fixed, parent forearm_skin_root_cell_link, child forearm_ring_4_link_3, origin xyz=0.0365 -0.0255 0.2122 rpy=-1.6695 -1.4976 -2.1060, axis 0 0 1, limit lower=0 upper=0 effort=150.0 velocity=3.15
- added joint forearm_ring_4_joint_4: type fixed, parent forearm_skin_root_cell_link, child forearm_ring_4_link_4, origin xyz=0.014 -0.043 0.211 rpy=0.1949 -1.5010 1.7227, axis 0 0 1, limit lower=0 upper=0 effort=150.0 velocity=3.15
- added joint forearm_ring_4_joint_5: type fixed, parent forearm_skin_root_cell_link, child forearm_ring_4_link_5, origin xyz=-0.0127 -0.0445 0.2117 rpy=2.2710 -1.5265 -1.0597
- added joint forearm_ring_4_joint_6: type fixed, parent forearm_skin_root_cell_link, child forearm_ring_4_link_6, origin xyz=-0.0423 -0.001 0.2124 rpy=0.6104 -1.539 -0.6458
- added joint forearm_ring_4_joint_7: type fixed, parent forearm_skin_root_cell_link, child forearm_ring_4_link_7, origin xyz=-0.0348 -0.0271 0.2127 rpy=-1.270 -1.540 1.899
- added joint forearm_ring_5_joint_0: type fixed, parent forearm_skin_root_cell_link, child forearm_ring_5_link_0, origin xyz=-0.02313 0.03352 0.23674 rpy=2.83297311  -1.54208643 2.44288303, axis 0 0 1, limit lower=0 upper=0 effort=150.0 velocity=3.15
- added joint forearm_ring_5_joint_1: type fixed, parent forearm_skin_root_cell_link, child forearm_ring_5_link_1, origin xyz=-0.04032 -0.015129 0.23696 rpy=1.06341521  -1.48901494 -0.78506072, axis 0 0 1, limit lower=0 upper=0 effort=150.0 velocity=3.15
- added joint forearm_ring_5_joint_2: type fixed, parent forearm_skin_root_cell_link, child forearm_ring_5_link_2, origin xyz=-0.0254929 -0.0339481 0.2358651 rpy=2.262972 -1.487026 -1.356827, axis 0 0 1, limit lower=0 upper=0 effort=150.0 velocity=3.15
- added joint forearm_ring_5_joint_3: type fixed, parent forearm_skin_root_cell_link, child forearm_ring_5_link_3, origin xyz=0.0004 -0.0441 0.23518 rpy=0.2035706 -1.5367411 1.35411575, axis 0 0 1, limit lower=0 upper=0 effort=150.0 velocity=3.15
- added joint forearm_ring_5_joint_4: type fixed, parent forearm_skin_root_cell_link, child forearm_ring_5_link_4, origin xyz=0.026086 -0.03677 0.23527 rpy=-2.34960077 -1.49847097 -1.75719079, axis 0 0 1, limit lower=0 upper=0 effort=150.0 velocity=3.15
- added joint forearm_ring_5_joint_5: type fixed, parent forearm_skin_root_cell_link, child forearm_ring_5_link_5, origin xyz=0.04277 -0.01486 0.23704 rpy=-2.16054646 -1.50515821 -1.31557256, axis 0 0 1, limit lower=0 upper=0 effort=150.0 velocity=3.15
- added joint forearm_ring_5_joint_6: type fixed, parent forearm_skin_root_cell_link, child forearm_ring_5_link_6, origin xyz=0.04285 0.01209 0.2382 rpy=-2.17682483 -1.51293455 -0.67460558, axis 0 0 1, limit lower=0 upper=0 effort=150.0 velocity=3.15
- added joint forearm_ring_5_joint_7: type fixed, parent forearm_skin_root_cell_link, child forearm_ring_5_link_7, origin xyz=0.02665 0.03505 0.23515 rpy=0.99763746 -1.51906704 3.11362853, axis 0 0 1, limit lower=0 upper=0 effort=150.0 velocity=3.15
- added joint forearm_skin_root_cell_joint: type fixed, parent forearm_link, child forearm_skin_root_cell_link, origin xyz=0.0 0.0 0.0 rpy=0.  0.  0., axis 0 0 1, limit lower=0 upper=0 effort=150.0 velocity=3.15

Commit message: Working changes on the real robot

File: urdf/skin.urdf.xacro (robot description, xacro)
@@ -132,5 +132,5 @@
 	  <parent link="forerarm_skin_root_cell_link"/>
 	  <child link="forerarm_skin_link_4"/>
-	  <origin xyz="0.026086 0.03677 0.23527" rpy="-2.34960077 -1.49847097 -1.75719079"/>
+	  <origin xyz="0.026086 -0.03677 0.23527" rpy="-2.34960077 -1.49847097 -1.75719079"/>
           <axis xyz="0 0 1" />
           <limit lower="0" upper="0" effort="150.0" velocity="3.15"/>

File: urdf/ur5_robot_with_ring_forearm.urdf (robot description, URDF)
Before this commit: robot ur5, 20 links, 19 joints
Joints:
- joint forerarm_skin_cell_joint_0: limit lower=-3.14159265 upper=3.14159265 effort=150.0 velocity=3.15 -> lower=0 upper=0 effort=150.0 velocity=3.15
- joint forerarm_skin_cell_joint_1: limit lower=-3.14159265 upper=3.14159265 effort=150.0 velocity=3.15 -> lower=0 upper=0 effort=150.0 velocity=3.15
- joint forerarm_skin_cell_joint_2: limit lower=-3.14159265 upper=3.14159265 effort=150.0 velocity=3.15 -> lower=0 upper=0 effort=150.0 velocity=3.15
- joint forerarm_skin_cell_joint_3: limit lower=-3.14159265 upper=3.14159265 effort=150.0 velocity=3.15 -> lower=0 upper=0 effort=150.0 velocity=3.15
- joint forerarm_skin_cell_joint_4: limit lower=-3.14159265 upper=3.14159265 effort=150.0 velocity=3.15 -> lower=0 upper=0 effort=150.0 velocity=3.15; origin xyz=0.026086 0.03677 0.23527 rpy=-2.34960077 -1.49847097 -1.75719079 -> xyz=0.026086 -0.03677 0.23527 rpy=-2.34960077 -1.49847097 -1.75719079
- joint forerarm_skin_cell_joint_5: limit lower=-3.14159265 upper=3.14159265 effort=150.0 velocity=3.15 -> lower=0 upper=0 effort=150.0 velocity=3.15
- joint forerarm_skin_cell_joint_6: limit lower=-3.14159265 upper=3.14159265 effort=150.0 velocity=3.15 -> lower=0 upper=0 effort=150.0 velocity=3.15
- joint forerarm_skin_cell_joint_7: limit lower=-3.14159265 upper=3.14159265 effort=150.0 velocity=3.15 -> lower=0 upper=0 effort=150.0 velocity=3.15
